File: Electrical circuits/Main circuit/Main circuit.kicad_sch (KiCad schematic)
At the start: 5 parts, among them U1 MOUDLE-SEEEDUINO-XIAO-ESP32C3, U2 DFPlayer Mini

Commit message: Made the final version of the circuit
Parts:
- added RV1, RV2: 100k, symbol Device:R_Potentiometer
- added SW1: Button, symbol Switch:SW_Push
Connections:
- net GND: now also RV1.3, RV2.3, SW1.2
- net at U1.1 (PA02_A0_D0): now also RV1.2
- net at U1.10 (PA5_A9_D9_MISO): now also SW1.1
- net +3.3V: now reaches U1.12 (3V3)
- net +3.3V: now also U2. (VCC), RV1.1, RV2.1
- net at U1.2 (PA4_A1_D1): now also RV2.2
- net +5V: no longer names the net of U1.14 (5V)
- net +5V: no longer U2. (VCC)
- no-connect marks 19 -> 17
Other:
- moved on the sheet: R1, R2
